File: dmf CTRL board/dmfboard.sch (EAGLE design)
At the start: 103 parts

Commit message: changed the control board circuit, added jumper pins & one extra inverter
Parts:
- removed MAX2: MAX7300, DMFlib:MAX7300
- removed R53, R54, R55, R56, R57, R58, R59, R60, R61, R62, R63, R64, R65, R66, R67: 1k, resistor:R-US_M0805
- removed U$1, U$2, U$22, U$23, U$24, U$25, U$26, U$27, U$28, U$29, U$30, U$31, U$32, U$33, U$34, U$35, U$36, U$37, U$38, U$39, U$40, U$41, U$42, U$43, U$44, U$45, U$46, U$47, U$48, U$49: AQW21, DMFlib:AQW21
- removed U$13, U$14, U$15, U$16, U$17: 74AC540, DMFlib:74AC540
- removed U$50: S5750_20_ND40PIN_CONNECTOR, DMFlib:S5750_20_ND40PIN_CONNECTOR
- added CONX1: S5750_20_ND40PIN_CONNECTOR, DMFlib:S5750_20_ND40PIN_CONNECTOR
- added IX1, IX2, IX3, IX4, IX5, IX6: 74AC540, DMFlib:74AC540
- added J1, J2, J3, J4: JUMPER, DMFlib:JUMPER
- added MX2: MAX7300, DMFlib:MAX7300
- added PX11, PX12, PX13, PX14, PX15, PX16, PX17, PX18, PX19, PX20, PX21, PX22, PX23, PX24, PX25, PX26, PX27, PX28, PX29, PX30, PX31, PX32, PX33, PX34, PX35, PX36, PX37, PX38, PX39, PX40: AQW21, DMFlib:AQW21
- added R11, R12, R13, R14, R15, R16, R17, R18, R19, R20, R6, R7, R8, R9: 1k, resistor:R-US_M0805
- added R3: 39K, resistor:R-US_M0805
- added R4: 1K, resistor:R-US_M0805
- R1: value 1K -> 4.7K
- R10: value 39K -> 1k
- R21, R22, R23, R24: value 1K -> 1k
- R25, R27: value 4.7K -> 1k
- R26: value 4.7K -> 1K
- R47, R48, R52: value 1k -> 1K
- R49: value 1k -> 39K
- R5: value 39K -> 1K
- R50, R51: value 1k -> 4.7K
- renumbered MAX1 to MX1, U$10 to PX2, U$11 to PX1, U$12 to PX10, U$3 to PX3, U$4 to PX4, U$5 to PX5, U$51 to 5V, U$52 to AMP, U$6 to PX6, U$7 to PX7, U$8 to PX8, U$9 to PX9
Connections:
- removed net N$113: MAX2.P12, R59.1, U$16.I7
- removed net N$122: MAX2.P14, R61.1, U$15.I1
- new net AD0: J1.1, J1.2, J1.3, J1.4, MX1.AD0
- new net AD00: J3.1, J3.2, J3.3, J3.4, MX2.AD0
- new net AD1: J2.1, J2.2, J2.3, J2.4, MX1.AD1
- new net AD11: J4.1, J4.2, J4.3, J4.4, MX2.AD1
- new net N$11: IX4.I1, MX2.P14, R40.1
- new net N$18: IX5.I7, MX2.P12, R38.1
- new net N$8: IX6.VCC, R52.1
- net AMP: now also PX1.P$8, PX10.P$8, PX11.P$8, PX12.P$8, PX13.P$8, PX14.P$8, PX15.P$8, PX16.P$8, PX17.P$8, PX18.P$8, PX19.P$8, PX2.P$8, PX20.P$8, PX21.P$8, PX22.P$8, PX23.P$8, PX24.P$8, PX25.P$8, PX26.P$8, PX27.P$8, PX28.P$8, PX29.P$8, PX3.P$8, PX30.P$8, PX31.P$8, PX32.P$8, PX33.P$8, PX34.P$8, PX35.P$8, PX36.P$8, PX37.P$8, PX38.P$8, PX39.P$8, PX4.P$8, PX40.P$8, PX5.P$8, PX6.P$8, PX7.P$8, PX8.P$8, PX9.P$8; no longer PX1.P$5, PX10.P$5, PX2.P$5, PX3.P$5, PX4.P$5, PX5.P$5, PX6.P$5, PX7.P$5, PX8.P$5, PX9.P$5, U$1.P$5, U$2.P$5, U$22.P$5, U$23.P$5, U$24.P$5, U$25.P$5, U$26.P$5, U$27.P$5, U$28.P$5, U$29.P$5, U$30.P$5, U$31.P$5, U$32.P$5, U$33.P$5, U$34.P$5, U$35.P$5, U$36.P$5, U$37.P$5, U$38.P$5, U$39.P$5, U$40.P$5, U$41.P$5, U$42.P$5, U$43.P$5, U$44.P$5, U$45.P$5, U$46.P$5, U$47.P$5, U$48.P$5, U$49.P$5
- net E1: now also CONX1.P$1; no longer U$50.P$1
- net E10: now also CONX1.P$10; no longer U$50.P$10
- net E11: now also CONX1.P$11, PX11.P$6, PX11.P$7; no longer U$28.P$6, U$28.P$7, U$50.P$11
- net E12: now also CONX1.P$12, PX12.P$6, PX12.P$7; no longer U$27.P$6, U$27.P$7, U$50.P$12
- net E13: now also CONX1.P$13, PX13.P$6, PX13.P$7; no longer U$1.P$6, U$1.P$7, U$50.P$13
- net E14: now also CONX1.P$14, PX14.P$6, PX14.P$7; no longer U$2.P$6, U$2.P$7, U$50.P$14
- net E15: now also CONX1.P$15, PX15.P$6, PX15.P$7; no longer U$22.P$6, U$22.P$7, U$50.P$15
- net E16: now also CONX1.P$16, PX16.P$6, PX16.P$7; no longer U$23.P$6, U$23.P$7, U$50.P$16
- net E17: now also CONX1.P$17, PX17.P$6, PX17.P$7; no longer U$24.P$6, U$24.P$7, U$50.P$17
- net E18: now also CONX1.P$18, PX18.P$6, PX18.P$7; no longer U$25.P$6, U$25.P$7, U$50.P$18
- net E19: now also CONX1.P$19, PX19.P$6, PX19.P$7; no longer U$26.P$6, U$26.P$7, U$50.P$19
- net E2: now also CONX1.P$2; no longer U$50.P$2
- net E20: now also CONX1.P$20, PX20.P$6, PX20.P$7; no longer U$29.P$6, U$29.P$7, U$50.P$20
- net E21: now also CONX1.P$21, PX21.P$6, PX21.P$7; no longer U$38.P$6, U$38.P$7, U$50.P$21
- net E22: now also CONX1.P$22, PX22.P$6, PX22.P$7; no longer U$37.P$6, U$37.P$7, U$50.P$22
- net E23: now also CONX1.P$23, PX23.P$6, PX23.P$7; no longer U$30.P$6, U$30.P$7, U$50.P$23
- net E24: now also CONX1.P$24, PX24.P$6, PX24.P$7; no longer U$31.P$6, U$31.P$7, U$50.P$24
- net E25: now also CONX1.P$25, PX25.P$6, PX25.P$7; no longer U$32.P$6, U$32.P$7, U$50.P$25
- net E26: now also CONX1.P$26, PX26.P$6, PX26.P$7; no longer U$33.P$6, U$33.P$7, U$50.P$26
- net E27: now also CONX1.P$27, PX27.P$6, PX27.P$7; no longer U$34.P$6, U$34.P$7, U$50.P$27
- net E28: now also CONX1.P$28, PX28.P$6, PX28.P$7; no longer U$35.P$6, U$35.P$7, U$50.P$28
- net E29: now also CONX1.P$29, PX29.P$6, PX29.P$7; no longer U$36.P$6, U$36.P$7, U$50.P$29
- net E3: now also CONX1.P$3; no longer U$50.P$3
- net E30: now also CONX1.P$30, PX30.P$6, PX30.P$7; no longer U$39.P$6, U$39.P$7, U$50.P$30
- net E31: now also CONX1.P$31, PX31.P$6, PX31.P$7; no longer U$48.P$6, U$48.P$7, U$50.P$31
- net E32: now also CONX1.P$32, PX32.P$6, PX32.P$7; no longer U$47.P$6, U$47.P$7, U$50.P$32
- net E33: now also CONX1.P$33, PX33.P$6, PX33.P$7; no longer U$40.P$6, U$40.P$7, U$50.P$33
- net E34: now also CONX1.P$34, PX34.P$6, PX34.P$7; no longer U$41.P$6, U$41.P$7, U$50.P$34
- net E35: now also CONX1.P$35, PX35.P$6, PX35.P$7; no longer U$42.P$6, U$42.P$7, U$50.P$35
- net E36: now also CONX1.P$36, PX36.P$6, PX36.P$7; no longer U$43.P$6, U$43.P$7, U$50.P$36
- net E37: now also CONX1.P$37, PX37.P$6, PX37.P$7; no longer U$44.P$6, U$44.P$7, U$50.P$37
- net E38: now also CONX1.P$38, PX38.P$6, PX38.P$7; no longer U$45.P$6, U$45.P$7, U$50.P$38
- net E39: now also CONX1.P$39, PX39.P$6, PX39.P$7; no longer U$46.P$6, U$46.P$7, U$50.P$39
- net E4: now also CONX1.P$4; no longer U$50.P$4
- net E40: now also CONX1.P$40, PX40.P$6, PX40.P$7; no longer U$49.P$6, U$49.P$7, U$50.P$40
- net E5: now also CONX1.P$5; no longer U$50.P$5
- net E6: now also CONX1.P$6; no longer U$50.P$6
- net E7: now also CONX1.P$7; no longer U$50.P$7
- net E8: now also CONX1.P$8; no longer U$50.P$8
- net E9: now also CONX1.P$9; no longer U$50.P$9
- net GND: now also IX1.GND, IX1.OE1, IX1.OE2, IX2.GND, IX2.OE1, IX2.OE2, IX3.GND, IX3.OE1, IX3.OE2, IX4.GND, IX4.OE1, IX4.OE2, IX5.GND, IX5.OE1, IX5.OE2, IX6.GND, IX6.OE1, IX6.OE2, J1.GND, J2.GND, J3.GND, J4.GND, MX2.GND, MX2.GND2, PX11.P$2, PX11.P$4, PX12.P$2, PX12.P$4, PX13.P$2, PX13.P$4, PX14.P$2, PX14.P$4, PX15.P$2, PX15.P$4, PX16.P$2, PX16.P$4, PX17.P$2, PX17.P$4, PX18.P$2, PX18.P$4, PX19.P$2, PX19.P$4, PX20.P$2, PX20.P$4, PX21.P$2, PX21.P$4, PX22.P$2, PX22.P$4, PX23.P$2, PX23.P$4, PX24.P$2, PX24.P$4, PX25.P$2, PX25.P$4, PX26.P$2, PX26.P$4, PX27.P$2, PX27.P$4, PX28.P$2, PX28.P$4, PX29.P$2, PX29.P$4, PX30.P$2, PX30.P$4, PX31.P$2, PX31.P$4, PX32.P$2, PX32.P$4, PX33.P$2, PX33.P$4, PX34.P$2, PX34.P$4, PX35.P$2, PX35.P$4, PX36.P$2, PX36.P$4, PX37.P$2, PX37.P$4, PX38.P$2, PX38.P$4, PX39.P$2, PX39.P$4, PX40.P$2, PX40.P$4, R3.1, R49.1; no longer MAX2.AD1, MAX2.GND, MAX2.GND2, MX1.AD0, MX1.AD1, R10.1, R5.1, U$1.P$2, U$1.P$4, U$13.GND, U$13.OE1, U$13.OE2, U$14.GND, U$14.OE1, U$14.OE2, U$15.GND, U$15.OE1, U$15.OE2, U$16.GND, U$16.OE1, U$16.OE2, U$17.GND, U$17.OE1, U$17.OE2, U$2.P$2, U$2.P$4, U$22.P$2, U$22.P$4, U$23.P$2, U$23.P$4, U$24.P$2, U$24.P$4, U$25.P$2, U$25.P$4, U$26.P$2, U$26.P$4, U$27.P$2, U$27.P$4, U$28.P$2, U$28.P$4, U$29.P$2, U$29.P$4, U$30.P$2, U$30.P$4, U$31.P$2, U$31.P$4, U$32.P$2, U$32.P$4, U$33.P$2, U$33.P$4, U$34.P$2, U$34.P$4, U$35.P$2, U$35.P$4, U$36.P$2, U$36.P$4, U$37.P$2, U$37.P$4, U$38.P$2, U$38.P$4, U$39.P$2, U$39.P$4, U$40.P$2, U$40.P$4, U$41.P$2, U$41.P$4, U$42.P$2, U$42.P$4, U$43.P$2, U$43.P$4, U$44.P$2, U$44.P$4, U$45.P$2, U$45.P$4, U$46.P$2, U$46.P$4, U$47.P$2, U$47.P$4, U$48.P$2, U$48.P$4, U$49.P$2, U$49.P$4
- net GND_AMP: now also PX1.P$5, PX10.P$5, PX11.P$5, PX12.P$5, PX13.P$5, PX14.P$5, PX15.P$5, PX16.P$5, PX17.P$5, PX18.P$5, PX19.P$5, PX2.P$5, PX20.P$5, PX21.P$5, PX22.P$5, PX23.P$5, PX24.P$5, PX25.P$5, PX26.P$5, PX27.P$5, PX28.P$5, PX29.P$5, PX3.P$5, PX30.P$5, PX31.P$5, PX32.P$5, PX33.P$5, PX34.P$5, PX35.P$5, PX36.P$5, PX37.P$5, PX38.P$5, PX39.P$5, PX4.P$5, PX40.P$5, PX5.P$5, PX6.P$5, PX7.P$5, PX8.P$5, PX9.P$5; no longer PX1.P$8, PX10.P$8, PX2.P$8, PX3.P$8, PX4.P$8, PX5.P$8, PX6.P$8, PX7.P$8, PX8.P$8, PX9.P$8, U$1.P$8, U$2.P$8, U$22.P$8, U$23.P$8, U$24.P$8, U$25.P$8, U$26.P$8, U$27.P$8, U$28.P$8, U$29.P$8, U$30.P$8, U$31.P$8, U$32.P$8, U$33.P$8, U$34.P$8, U$35.P$8, U$36.P$8, U$37.P$8, U$38.P$8, U$39.P$8, U$40.P$8, U$41.P$8, U$42.P$8, U$43.P$8, U$44.P$8, U$45.P$8, U$46.P$8, U$47.P$8, U$48.P$8, U$49.P$8
- net N$1: now also MX2.ISET, R49.2; no longer MAX2.ISET, R5.2
- net N$103: now also PX31.P$1, R37.2; no longer R58.2, U$48.P$1
- net N$104: now also PX32.P$1, R38.2; no longer R59.2, U$47.P$1
- net N$105: now also PX33.P$1, R39.2; no longer R60.2, U$40.P$1
- net N$106: now also PX34.P$1, R40.2; no longer R61.2, U$41.P$1
- net N$107: now also PX35.P$1, R41.2; no longer R62.2, U$42.P$1
- net N$108: now also PX36.P$1, R42.2; no longer R63.2, U$43.P$1
- net N$109: now also PX37.P$1, R43.2; no longer R64.2, U$44.P$1
- net N$110: now also PX38.P$1, R44.2; no longer R65.2, U$45.P$1
- net N$111: now also PX39.P$1, R45.2; no longer R66.2, U$46.P$1
- net N$112: now also PX40.P$1, R46.2; no longer R67.2, U$49.P$1
- net N$114: now also IX5.I1, MX2.P6, R32.1; no longer MAX2.P6, R53.1, U$16.I1
- net N$115: now also IX5.I2, MX2.P7, R33.1; no longer MAX2.P7, R54.1, U$16.I2
- net N$116: now also IX5.I3, MX2.P8, R34.1; no longer MAX2.P8, R55.1, U$16.I3
- net N$117: now also IX5.I4, MX2.P9, R35.1; no longer MAX2.P9, R56.1, U$16.I4
- net N$118: now also IX5.I5, MX2.P10, R36.1; no longer MAX2.P10, R57.1, U$16.I5
- net N$119: now also IX5.I6, MX2.P11, R37.1; no longer MAX2.P11, R58.1, U$16.I6
- net N$120: now also IX4.I2, MX2.P15, R41.1; no longer MAX2.P15, R62.1, U$15.I2
- net N$121: now also IX4.I0, MX2.P13, R39.1; no longer MAX2.P13, R60.1, U$15.I0
- net N$123: now also IX4.I3, MX2.P16, R42.1; no longer MAX2.P16, R63.1, U$15.I3
- net N$124: now also IX4.I4, MX2.P17, R43.1; no longer MAX2.P17, R64.1, U$15.I4
- net N$125: now also IX4.I5, MX2.P18, R44.1; no longer MAX2.P18, R65.1, U$15.I5
- net N$126: now also IX4.I6, MX2.P19, R45.1; no longer MAX2.P19, R66.1, U$15.I6
- net N$127: now also IX4.I7, MX2.P20, R46.1; no longer MAX2.P20, R67.1, U$15.I7
- net N$128: now also IX6.I0, MX2.P1, R27.1; no longer MAX2.P1, R48.1, U$14.I7
- net N$129: now also IX6.I1, MX2.P2, R28.1; no longer MAX2.P2, R49.1, U$14.I6
- net N$130: now also IX6.I2, MX2.P3, R29.1; no longer MAX2.P3, R50.1, U$14.I5
- net N$131: now also IX6.I3, MX2.P4, R30.1; no longer MAX2.P4, R51.1, U$14.I4
- net N$2: now also R3.2; no longer R10.2
- net N$28: now also R15.2; no longer R37.2
- net N$29: now also R14.2; no longer R36.2
- net N$3: now also IX1.VCC, R4.1; no longer R1.1, U$17.VCC
- net N$30: now also R13.2; no longer R35.2
- net N$31: now also R12.2; no longer R34.2
- net N$32: now also R11.2; no longer R33.2
- net N$33: now also R10.2; no longer R32.2
- net N$34: now also R9.2; no longer R31.2
- net N$35: now also R8.2; no longer R30.2
- net N$36: now also R7.2; no longer R29.2
- net N$37: now also R6.2; no longer R28.2
- net N$38: now also PX11.P$1, R16.2; no longer R38.2, U$28.P$1
- net N$39: now also PX12.P$1, R17.2; no longer R39.2, U$27.P$1
- net N$4: now also IX2.VCC, R5.1; no longer R21.1, U$13.VCC
- net N$40: now also PX13.P$1, R18.2; no longer R40.2, U$1.P$1
- net N$41: now also PX14.P$1, R19.2; no longer R41.2, U$2.P$1
- net N$42: now also PX15.P$1, R20.2; no longer R42.2, U$22.P$1
- net N$43: now also PX16.P$1, R21.2; no longer R43.2, U$23.P$1
- net N$44: now also PX17.P$1, R22.2; no longer R44.2, U$24.P$1
- net N$45: now also PX18.P$1, R23.2; no longer R45.2, U$25.P$1
- net N$46: now also PX19.P$1, R24.2; no longer R46.2, U$26.P$1
- net N$47: now also PX20.P$1, R25.2; no longer R47.2, U$29.P$1
- net N$48: now also IX1.I0, R6.1; no longer R28.1, U$17.I0
- net N$5: now also IX3.VCC, R26.1; no longer R22.1, U$14.VCC
- net N$50: now also IX1.I2, R8.1; no longer R30.1, U$17.I2
- net N$51: now also IX1.I3, R9.1; no longer R31.1, U$17.I3
- net N$52: now also IX1.I4, R10.1; no longer R32.1, U$17.I4
- net N$53: now also IX1.I5, R11.1; no longer R33.1, U$17.I5
- net N$54: now also IX1.I6, R12.1; no longer R34.1, U$17.I6
- net N$55: now also IX1.I7, R13.1; no longer R35.1, U$17.I7
- net N$56: now also IX2.I0, R14.1; no longer R36.1, U$13.I0
- net N$57: now also IX2.I1, R15.1; no longer R37.1, U$13.I1
- net N$58: now also IX2.I2, R16.1; no longer R38.1, U$13.I2
- net N$59: now also IX2.I3, R17.1; no longer R39.1, U$13.I3
- net N$6: now also IX4.VCC, R47.1; no longer R23.1, U$15.VCC
- net N$60: now also IX2.I4, R18.1; no longer R40.1, U$13.I4
- net N$61: now also IX2.I5, R19.1; no longer R41.1, U$13.I5
- net N$62: now also IX2.I6, R20.1; no longer R42.1, U$13.I6
- net N$63: now also IX2.I7, R21.1; no longer R43.1, U$13.I7
- net N$64: now also IX3.I0, R22.1; no longer R44.1, U$14.I0
- net N$65: now also IX3.I1, R23.1; no longer R45.1, U$14.I1
- net N$66: now also IX3.I2, R24.1; no longer R46.1, U$14.I2
- net N$67: now also IX3.I3, R25.1; no longer R47.1, U$14.I3
- net N$68: now also IX1.I1, R7.1; no longer R29.1, U$17.I1
- net N$7: now also IX5.VCC, R48.1; no longer R24.1, U$16.VCC
- net N$82: now also PX21.P$1, R27.2; no longer R48.2, U$38.P$1
- net N$83: now also PX22.P$1, R28.2; no longer R49.2, U$37.P$1
- net N$84: now also PX23.P$1, R29.2; no longer R50.2, U$30.P$1
- net N$85: now also PX24.P$1, R30.2; no longer R51.2, U$31.P$1
- net N$86: now also PX25.P$1, R31.2; no longer R52.2, U$32.P$1
- net N$87: now also PX26.P$1, R32.2; no longer R53.2, U$33.P$1
- net N$88: now also PX27.P$1, R33.2; no longer R54.2, U$34.P$1
- net N$89: now also PX28.P$1, R34.2; no longer R55.2, U$35.P$1
- net N$90: now also PX29.P$1, R35.2; no longer R56.2, U$36.P$1
- net N$91: now also PX30.P$1, R36.2; no longer R57.2, U$39.P$1
- net N$92: now also IX5.I0, MX2.P5, R31.1; no longer MAX2.P5, R52.1, U$16.I0
- net O0: now also IX1.O0; no longer U$17.O0
- net O1: now also IX1.O1; no longer U$17.O1
- net O10: now also IX2.O2, PX11.P$3; no longer U$13.O2, U$28.P$3
- net O11: now also IX2.O3, PX12.P$3; no longer U$13.O3, U$27.P$3
- net O12: now also IX2.O4, PX13.P$3; no longer U$1.P$3, U$13.O4
- net O13: now also IX2.O5, PX14.P$3; no longer U$13.O5, U$2.P$3
- net O14: now also IX2.O6, PX15.P$3; no longer U$13.O6, U$22.P$3
- net O15: now also IX2.O7, PX16.P$3; no longer U$13.O7, U$23.P$3
- net O16: now also IX3.O0, PX17.P$3; no longer U$14.O0, U$24.P$3
- net O17: now also IX3.O1, PX18.P$3; no longer U$14.O1, U$25.P$3
- net O18: now also IX3.O2, PX19.P$3; no longer U$14.O2, U$26.P$3
- net O19: now also IX3.O3, PX20.P$3; no longer U$14.O3, U$29.P$3
- net O2: now also IX1.O2; no longer U$17.O2
- net O20: now also IX6.O0, PX21.P$3; no longer U$14.O4, U$38.P$3
- net O21: now also IX6.O1, PX22.P$3; no longer U$14.O5, U$37.P$3
- net O22: now also IX6.O2, PX23.P$3; no longer U$14.O6, U$30.P$3
- net O23: now also IX6.O3, PX24.P$3; no longer U$14.O7, U$31.P$3
- net O24: now also IX5.O0, PX25.P$3; no longer U$16.O0, U$32.P$3
- net O25: now also IX5.O1, PX26.P$3; no longer U$16.O1, U$33.P$3
- net O26: now also IX5.O2, PX27.P$3; no longer U$16.O2, U$34.P$3
- net O27: now also IX5.O3, PX28.P$3; no longer U$16.O3, U$35.P$3
- net O28: now also IX5.O4, PX29.P$3; no longer U$16.O4, U$36.P$3
- net O29: now also IX5.O5, PX30.P$3; no longer U$16.O5, U$39.P$3
- net O3: now also IX1.O3; no longer U$17.O3
- net O30: now also IX5.O6, PX31.P$3; no longer U$16.O6, U$48.P$3
- net O31: now also IX5.O7, PX32.P$3; no longer U$16.O7, U$47.P$3
- net O32: now also IX4.O0, PX33.P$3; no longer U$15.O0, U$40.P$3
- net O33: now also IX4.O1, PX34.P$3; no longer U$15.O1, U$41.P$3
- net O34: now also IX4.O2, PX35.P$3; no longer U$15.O2, U$42.P$3
- net O35: now also IX4.O3, PX36.P$3; no longer U$15.O3, U$43.P$3
- net O36: now also IX4.O4, PX37.P$3; no longer U$15.O4, U$44.P$3
- net O37: now also IX4.O5, PX38.P$3; no longer U$15.O5, U$45.P$3
- net O38: now also IX4.O6, PX39.P$3; no longer U$15.O6, U$46.P$3
- net O39: now also IX4.O7, PX40.P$3; no longer U$15.O7, U$49.P$3
- net O4: now also IX1.O4; no longer U$17.O4
- net O5: now also IX1.O5; no longer U$17.O5
- net O6: now also IX1.O6; no longer U$17.O6
- net O7: now also IX1.O7; no longer U$17.O7
- net O8: now also IX2.O0; no longer U$13.O0
- net O9: now also IX2.O1; no longer U$13.O1
- net SCL: now also J1.SCL, J2.SCL, J3.SCL, J4.SCL, MX2.SCL, R2.2, R51.2; no longer MAX2.SCL, R25.2, R26.2
- net SDA: now also J1.SDA, J2.SDA, J3.SDA, J4.SDA, MX2.SDA, R1.2, R50.2; no longer MAX2.SDA, R2.2, R27.2
- net VDD: now also J1.V+, J2.V+, J3.V+, J4.V+, MX2.V+, R1.1, R26.2, R4.2, R47.2, R48.2, R5.2, R50.1, R51.1, R52.2; no longer MAX2.AD0, MAX2.V+, R1.2, R21.2, R22.2, R23.2, R24.2, R25.1, R26.1, R27.1
Other:
- note added: "MAX1 jumper"
- note added: "MAX2 jumper"
- note removed: "Address x40"
- note removed: "Address x41"
- moved on the sheet: R1, R10, R2, R21, R22, R23, R24, R25, R26, R27, R28, R29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
